Commit message: calibrating cameras

File: pepper_description/urdf/pepper1.0_generated_urdf/pepper.urdf (robot description, URDF)
Before this commit: robot JulietteY20MP, 83 links, 82 joints
Joints:
- joint CameraDepth_optical_frame_fixedjoint: origin xyz=0 0 0 rpy=-1.57079632679 0 -1.57079632679 -> xyz=0 0 0 rpy=-1.5936 -0.0161345 -1.57777
- joint CameraDepth_sensor_fixedjoint: origin xyz=0.05138 0.039 0.1194 rpy=0 0 0 -> xyz=0.0708098 0.02 0.118115 rpy=0 0 0

File: pepper_description/urdf/pepper1.0_generated_urdf/pepper_sensors.xacro (robot description, xacro)
@@ -21,5 +21,5 @@
 		<parent link="CameraDepth_frame"/>
 		<child link="CameraDepth_optical_frame"/>
-		<origin rpy="-1.57079632679 0 -1.57079632679" xyz="0 0 0"/>
+		<origin rpy="-1.5936 -0.0161345 -1.57777" xyz="0 0 0"/>
 	</joint>
 	<link name="LHandTouchBack_frame"/>
@@ -118,5 +118,5 @@
 		<parent link="Head"/>
 		<child link="CameraDepth_frame"/>
-		<origin rpy="0 0 0" xyz="0.05138 0.039 0.1194"/>
+		<origin rpy="0 0 0" xyz="0.0708098 0.02 0.118115"/>
 		<axis xyz="0 0 0"/>
 	</joint>
